File: pcb/tc69.kicad_pcb (KiCad board)
At the start: 2 copper layers, 96 parts, among them SW1 ESC, SW10 LWIN, SW11 2, SW12 W, SW13 A, SW14 Z, SW16 3, SW17 E, SW18 S, SW19 X, SW2 TAB, SW20 LALT, SW21 4, SW22 R, SW23 D, SW24 C, SW26 5, SW27 T, SW28 F, SW29 V, SW3 CAPS, SW30 LSPC, SW31 6, SW32 Y, SW33 G, SW34 B, SW36 7, SW37 U, SW38 H, SW39 N, SW41 8, SW42 I, SW43 J, SW44 M, SW45 RSPC, SW46 9, SW47 O, SW48 K, SW49 COMMA, SW5 LCTRL, SW51 0, SW52 P, SW53 L, SW54 DOT, SW55 RALT, SW56 MINUS, SW57 LBRC, SW58 SCLN, SW59 SLSH, SW6 1, SW60 RWIN, SW61 EQUAL, SW62 RBRC, SW63 QUOTE, SW65 APP, SW66 BS, SW68 ENTER, SW69 RSHFT, SW7 Q, SW70 LEFT, SW72 BSLSH, SW74 UP, SW75 DOWN, SW76 HOME, SW77 PGUP, SW78 PGDN, SW79 END, SW80 RIGHT, SW9 LSHFT, U1 SeeeduinoXIAO, U2 CD74HC4067SM, U3 TLV9051

Commit message: partly routed
Parts:
- moved C2 88.1 mm to (92.3, -4.05), turned to 90 degrees
- moved R3 87.4 mm to (94.1, -4.40)
- moved R1 84.2 mm to (101.8, -9.30), turned to 90 degrees
- moved R2 80.4 mm to (104.0, -9.25), turned to 90 degrees
- moved U3 79.6 mm to (103.0, -5.95), turned to 0 degrees
- moved C4 79.2 mm to (103.1, -3.57), turned to 0 degrees
- moved C3 78.2 mm to (106.0, -9.05), turned to 90 degrees
- moved U2 37.5 mm to (147.0, 33.3)
- moved U1 32.1 mm to (155.9, 25.6)
- moved C1 21.4 mm to (114.9, 13.6), turned to 90 degrees
- moved R4 5.16 mm to (5.95, 38.1)
- moved R6 5.02 mm to (44.1, 38.1)
- moved R17 4.92 mm to (253.6, 38.1)
- moved R5 4.91 mm to (25.0, 38.1)
- moved R19 4.71 mm to (291.7, 38.1)
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Routing:
- net col1: track 0.00 -> 237.2 mm, vias 0 -> 4
- net col2: track 0.00 -> 203.8 mm, vias 0 -> 4
- net col3: track 0.00 -> 138.5 mm, vias 0 -> 4
- net col16: track 0.00 -> 103.2 mm, vias 0 -> 1
- net col4: track 0.00 -> 95.3 mm, vias 0 -> 5
- net col12: track 0.00 -> 66.4 mm
- net col5: track 0.00 -> 65.9 mm, vias 0 -> 4
- net col14: track 0.00 -> 56.9 mm
- net col13: track 0.00 -> 51.1 mm
- net col15: track 0.00 -> 49.1 mm
- net col11: track 0.00 -> 46.7 mm
- net col6: track 0.00 -> 45.8 mm, vias 0 -> 4
- net col10: track 0.00 -> 26.9 mm
- net col7: track 0.00 -> 25.7 mm, vias 0 -> 1
- net S0: track 20.2 -> 0.00 mm
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Other:
- net class Power added: clearance 0.2, trace_width 0.5, via_dia 0.8, via_drill 0.4

Commit message: wire a bit
Parts:
- added C5: 100n, Capacitor_SMD:C_0402_1005Metric, B.Cu at (72.7, 36.3)
- added C6: 100n, Capacitor_SMD:C_0402_1005Metric, B.Cu at (225.0, 36.3)
- added U4: 4051, Package_SO:SOIC-16_3.9x9.9mm_P1.27mm, B.Cu at (70.8, 30.4)
- added U5: 4051, Package_SO:SOIC-16_3.9x9.9mm_P1.27mm, B.Cu at (223.2, 30.4)
- U2: value CD74HC4067SM -> 74AHC1G04; footprint Package_SO:SSOP-24_5.3x8.2mm_P0.65mm -> Package_TO_SOT_SMD:SOT-23-5
- moved C1 51.2 mm to (164.3, 26.9)
- moved C3 46.1 mm to (129.8, 30.5)
- moved R11 46.0 mm to (93.5, 34.2), turned to 270 degrees
- moved R19 46.0 mm to (245.9, 34.2), turned to 270 degrees
- moved R3 43.2 mm to (119.7, 30.4)
- moved U3 43.1 mm to (126.2, 30.4)
- moved R2 43.1 mm to (128.0, 26.5)
- moved R1 42.7 mm to (125.0, 26.6)
- moved R12 42.4 mm to (200.6, 34.2), turned to 270 degrees
- moved R4 42.4 mm to (48.2, 34.2), turned to 270 degrees
- moved C2 42.2 mm to (116.1, 30.8), turned to 270 degrees
- moved C4 39.3 mm to (122.6, 30.5), turned to 270 degrees
- moved R10 32.3 mm to (88.1, 34.8), turned to 270 degrees
- moved R18 32.3 mm to (240.5, 34.8), turned to 270 degrees
- moved R5 28.8 mm to (53.6, 34.8), turned to 270 degrees
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Connections:
- U1 pad 1: row1 -> S0
- U1 pad 2: row2 -> S1
- U1 pad 3: row3 -> S2
- U1 pad 4: row4 -> S3
- U1 pad 6: S3 -> row4
- U1 pad 7: S2 -> row3
- U1 pad 8: S1 -> row1
- U1 pad 9: S0 -> row2
- U2 pad 1: SENSE -> (no net)
- U2 pad 2: col8 -> S0
- U2 pad 3: col7 -> GND
- U2 pad 4: col6 -> IS0
- U2 pad 5: col5 -> +5V
Routing:
- net row2: track 0.00 -> 416.2 mm, vias 6 -> 25
- net row1: track 0.00 -> 306.0 mm, vias 5 -> 25
- net col1: track 237.2 -> 91.2 mm, vias 4 -> 3
- net col2: track 203.8 -> 72.6 mm, vias 4 -> 3
- net col16: track 103.2 -> 0.00 mm, vias 1 -> 3
- net col8: track 6.32 -> 94.6 mm, vias 0 -> 4
- net col3: track 138.5 -> 52.5 mm
- net col9: track 8.09 -> 92.2 mm, vias 0 -> 4
- net col14: track 56.9 -> 0.00 mm, vias 0 -> 2
- net col4: track 95.3 -> 38.9 mm
- net row3: track 0.00 -> 55.0 mm, vias 6 -> 14
- net +5V: track 53.3 -> 1.55 mm, vias 3 -> 0
- net col13: track 51.1 -> 0.00 mm, vias 0 -> 3
- net col12: track 66.4 -> 16.9 mm, vias 0 -> 3
- net col15: track 49.1 -> 0.00 mm, vias 0 -> 1
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