File: pcb/tc69.sch (KiCad schematic (older format))
At the start: 95 parts, among them SW1 ESC, SW10 LWIN, SW11 2, SW12 W, SW13 A, SW14 Z, SW16 3, SW17 E, SW18 S, SW19 X, SW2 TAB, SW20 LALT, SW21 4, SW22 R, SW23 D, SW24 C, SW26 5, SW27 T, SW28 F, SW29 V, SW3 CAPS, SW30 LSPC, SW31 6, SW32 Y, SW33 G, SW34 B, SW36 7, SW37 U, SW38 H, SW39 N, SW41 8, SW42 I, SW43 J, SW44 M, SW45 RSPC, SW46 9, SW47 O, SW48 K, SW49 COMMA, SW5 LCTRL, SW51 0, SW52 P, SW53 L, SW54 DOT, SW55 RALT, SW56 MINUS, SW57 LBRC, SW58 SCLN, SW59 SLSH, SW6 1, SW60 RWIN, SW61 EQUAL, SW62 RBRC, SW63 QUOTE, SW65 APP, SW66 BS, SW68 ENTER, SW69 RSHFT, SW7 Q, SW70 LEFT, SW72 BSLSH, SW74 UP, SW75 DOWN, SW76 HOME, SW77 PGUP, SW78 PGDN, SW79 END, SW80 RIGHT, SW9 LSHFT, U1 SeeeduinoXIAO, U2 CD74HC4067SM, U3 TLV9051

Commit message: wire a bit
Parts:
- removed U2: CD74HC4067SM, Package_SO:SSOP-24_5.3x8.2mm_P0.65mm, symbol 74xx:CD74HC4067SM
- added C5, C6: 100n, Capacitor_SMD:C_0402_1005Metric, symbol Device:C_Small
- added U2: 74AHC1G04, Package_TO_SOT_SMD:SOT-23-5, symbol 74xGxx:74AHC1G04
- added U4, U5: 4051, Package_SO:SOIC-16_3.9x9.9mm_P1.27mm, symbol 4xxx:4051
Connections:
- net +5V: now also C5.2, C6.2, U2.5 (VCC), U4.16 (VDD), U5.16 (VDD)
- net GND: now also C5.1, C6.1, U2.3 (GND), U4.7 (VEE), U4.8 (VSS), U5.7 (VEE), U5.8 (VSS)
- net S0: now also U1.1 (PA02_A0_D0), U2.2, U4.6 (Inh); no longer U1.9 (PA7_A8_D8_SCK)
- net S1: now also U1.2 (PA4_A1_D1), U4.11 (A), U5.11 (A); no longer U1.8 (PB09_A7_D7_RX)
- net S2: now also U1.3 (PA10_A2_D2), U4.10 (B), U5.10 (B); no longer U1.7 (PB08_A6_D6_TX)
- net S3: now also U1.4 (PA11_A3_D3), U4.9 (C), U5.9 (C); no longer U1.6 (PA9_A5_D5_SCL)
- net SENSE: now also U4.3 (X), U5.3 (X)
- net col1: now also U4.5 (X5)
- net col10: now also U5.4 (X7)
- net col11: now also U5.2 (X6)
- net col12: now also U5.1 (X4)
- net col13: now also U5.15 (X2)
- net col14: now also U5.14 (X1)
- net col15: now also U5.13 (X0)
- net col16: now also U5.12 (X3)
- net col2: now also U4.4 (X7)
- net col3: now also U4.2 (X6)
- net col4: now also U4.1 (X4)
- net col5: now also U4.15 (X2)
- net col6: now also U4.14 (X1)
- net col7: now also U4.13 (X0)
- net col8: now also U4.12 (X3)
- net col9: now also U5.5 (X5)
- net row1: now also U1.8 (PB09_A7_D7_RX); no longer U1.1 (PA02_A0_D0)
- net row2: now also U1.9 (PA7_A8_D8_SCK); no longer U1.2 (PA4_A1_D1)
- net row3: now also U1.7 (PB08_A6_D6_TX); no longer U1.3 (PA10_A2_D2)
- net row4: now also U1.6 (PA9_A5_D5_SCL); no longer U1.4 (PA11_A3_D3)
- new net IS0: U2.4, U5.6 (Inh)
Other:
- moved on the sheet: C1, C2, C3, C4, R1, R2, R3, U1, U3

Commit message: switch wired
Parts:
- removed SW63: QUOTE, lib:ecs_pad, symbol ec_sw:EC_SW
- added SW8: A, lib:ecs_pad, symbol ec_sw:EC_SW
- SW13: value A -> S
- SW18: value S -> D
- SW23: value D -> F
- SW28: value F -> G
- SW33: value G -> H
- SW38: value H -> J
- SW43: value J -> K
- SW48: value K -> L
- SW53: value L -> SCLN
- SW58: value SCLN -> QUOTE
Connections:
- net GND: now also SW8.3 (SG)
- net col2: now also SW8.2
- net row3: now also SW8.1
Changed lines of the file:
@@
 P 6550 3750
 F 0 "SW13" H 6583 3965 50  0000 C CNN
-F 1 "A" H 6583 3874 50  0000 C CNN
+F 1 "S" H 6583 3874 50  0000 C CNN
 F 2 "lib:ecs_pad" H 6550 3500 50  0001 C CNN
 F 3 "" H 6550 3500 50  0000 C CNN
@@
 L power:GND #PWR0124
 U 1 1 619841A1
-P 6600 3850
-F 0 "#PWR0124" H 6600 3600 50  0001 C CNN
-F 1 "GND" H 6605 3677 50  0001 C CNN
-F 2 "" H 6600 3850 50  0001 C CNN
-F 3 "" H 6600 3850 50  0001 C CNN
-	1    6600 3850
+P 6300 3850
+F 0 "#PWR0124" H 6300 3600 50  0001 C CNN
+F 1 "GND" H 6305 3677 50  0001 C CNN
+F 2 "" H 6300 3850 50  0001 C CNN
+F 3 "" H 6300 3850 50  0001 C CNN
+	1    6300 3850
 	1    0    0    -1
 $EndComp
@@
 	6700 2650 6700 3200
 Connection ~ 6700 3200
-Wire Wire Line
-	6700 3200 6700 3750
-Connection ~ 6700 3750
-Wire Wire Line
-	6700 3750 6700 4300
 $Comp
 L ec_sw:EC_SW SW16
@@
 P 8050 3750
 F 0 "SW38" H 8083 3965 50  0000 C CNN
-F 1 "H" H 8083 3874 50  0000 C CNN
+F 1 "J" H 8083 3874 50  0000 C CNN
 F 2 "lib:ecs_pad" H 8050 3500 50  0001 C CNN
 F 3 "" H 8050 3500 50  0000 C CNN
@@
 P 7750 3750
 F 0 "SW33" H 7783 3965 50  0000 C CNN
-F 1 "G" H 7783 3874 50  0000 C CNN
+F 1 "H" H 7783 3874 50  0000 C CNN
 F 2 "lib:ecs_pad" H 7750 3500 50  0001 C CNN
 F 3 "" H 7750 3500 50  0000 C CNN
@@
 P 7450 3750
 F 0 "SW28" H 7483 3965 50  0000 C CNN
-F 1 "F" H 7483 3874 50  0000 C CNN
+F 1 "G" H 7483 3874 50  0000 C CNN
 F 2 "lib:ecs_pad" H 7450 3500 50  0001 C CNN
 F 3 "" H 7450 3500 50  0000 C CNN
@@
 P 7150 3750
 F 0 "SW23" H 7183 3965 50  0000 C CNN
-F 1 "D" H 7183 3874 50  0000 C CNN
+F 1 "F" H 7183 3874 50  0000 C CNN
 F 2 "lib:ecs_pad" H 7150 3500 50  0001 C CNN
 F 3 "" H 7150 3500 50  0000 C CNN
@@
 P 6850 3750
 F 0 "SW18" H 6883 3965 50  0000 C CNN
-F 1 "S" H 6883 3874 50  0000 C CNN
+F 1 "D" H 6883 3874 50  0000 C CNN
 F 2 "lib:ecs_pad" H 6850 3500 50  0001 C CNN
 F 3 "" H 6850 3500 50  0000 C CNN
@@
 P 8350 3750
 F 0 "SW43" H 8383 3965 50  0000 C CNN
-F 1 "J" H 8383 3874 50  0000 C CNN
+F 1 "K" H 8383 3874 50  0000 C CNN
 F 2 "lib:ecs_pad" H 8350 3500 50  0001 C CNN
 F 3 "" H 8350 3500 50  0000 C CNN
@@
 P 8650 3750
 F 0 "SW48" H 8683 3965 50  0000 C CNN
-F 1 "K" H 8683 3874 50  0000 C CNN
+F 1 "L" H 8683 3874 50  0000 C CNN
 F 2 "lib:ecs_pad" H 8650 3500 50  0001 C CNN
 F 3 "" H 8650 3500 50  0000 C CNN
@@
 P 8950 3750
 F 0 "SW53" H 8983 3965 50  0000 C CNN
-F 1 "L" H 8983 3874 50  0000 C CNN
+F 1 "SCLN" H 8983 3874 50  0000 C CNN
 F 2 "lib:ecs_pad" H 8950 3500 50  0001 C CNN
 F 3 "" H 8950 3500 50  0000 C CNN
@@
 	1    0    0    -1
 $EndComp
-Connection ~ 9700 3750
-Wire Wire Line
-	9700 3200 9700 3750
 $Comp
 L power:GND #PWR0184
@@
 $EndComp
 $Comp
-L power:GND #PWR0186
-U 1 1 619EA8F8
-P 9600 3850
-F 0 "#PWR0186" H 9600 3600 50  0001 C CNN
-F 1 "GND" H 9605 3677 50  0001 C CNN
-F 2 "" H 9600 3850 50  0001 C CNN
-F 3 "" H 9600 3850 50  0001 C CNN
-	1    9600 3850
-	1    0    0    -1
-$EndComp
-$Comp
-L ec_sw:EC_SW SW63
-U 1 1 619EA8FE
-P 9550 3750
-F 0 "SW63" H 9583 3965 50  0000 C CNN
-F 1 "QUOTE" H 9583 3874 50  0000 C CNN
-F 2 "lib:ecs_pad" H 9550 3500 50  0001 C CNN
-F 3 "" H 9550 3500 50  0000 C CNN
-	1    9550 3750
-	1    0    0    -1
-$EndComp
-$Comp
 L power:GND #PWR0187
 U 1 1 619EA904
@@
 P 9250 3750
 F 0 "SW58" H 9283 3965 50  0000 C CNN
-F 1 "SCLN" H 9283 3874 50  0000 C CNN
+F 1 "QUOTE" H 9283 3874 50  0000 C CNN
 F 2 "lib:ecs_pad" H 9250 3500 50  0001 C CNN
 F 3 "" H 9250 3500 50  0000 C CNN
@@
 	5750 4000 5900 4000
 Connection ~ 5900 4000
-Connection ~ 6500 4000
-Wire Wire Line
-	6500 4000 6800 4000
 Connection ~ 6800 4000
 Wire Wire Line
@@
 	8900 4000 9200 4000
 Connection ~ 9200 4000
-Wire Wire Line
-	9200 4000 9500 4000
-Connection ~ 9500 4000
-Wire Wire Line
-	9500 4000 9800 4000
 Connection ~ 9800 4000
 Connection ~ 6200 4550
@@
 	6100 3750 6100 4850
 Wire Wire Line
-	5900 4000 6500 4000
-Wire Wire Line
-	6400 3200 6400 4300
+	6400 3200 6400 3750
 Wire Wire Line
 	6200 5100 6800 5100
@@
 Wire Wire Line
 	9200 4550 9800 4550
-Wire Wire Line
-	9700 3750 9700 4850
 Wire Wire Line
 	9800 2900 10400 2900
@@
 	2350 3500 1950 3500
 Connection ~ 2350 4700
+$Comp
+L ec_sw:EC_SW SW8
+U 1 1 61988E43
+P 6250 3750
+F 0 "SW8" H 6283 3965 50  0000 C CNN
+F 1 "A" H 6283 3874 50  0000 C CNN
+F 2 "lib:ecs_pad" H 6250 3500 50  0001 C CNN
+F 3 "" H 6250 3500 50  0000 C CNN
+	1    6250 3750
+	1    0    0    -1
+$EndComp
+Wire Wire Line
+	6700 3200 6700 3750
+Wire Wire Line
+	5900 4000 6200 4000
+$Comp
+L power:GND #PWR0186
+U 1 1 619947F9
+P 6600 3850
+F 0 "#PWR0186" H 6600 3600 50  0001 C CNN
+F 1 "GND" H 6605 3677 50  0001 C CNN
+F 2 "" H 6600 3850 50  0001 C CNN
+F 3 "" H 6600 3850 50  0001 C CNN
+	1    6600 3850
+	1    0    0    -1
+$EndComp
+Connection ~ 6500 4000
+Wire Wire Line
+	6500 4000 6800 4000
+Connection ~ 6700 3750
+Wire Wire Line
+	6700 3750 6700 4300
+Connection ~ 6200 4000
+Wire Wire Line
+	6200 4000 6500 4000
+Connection ~ 6400 3750
+Wire Wire Line
+	6400 3750 6400 4300
+Wire Wire Line
+	9200 4000 9800 4000
+Wire Wire Line
+	9700 3200 9700 4850
 $EndSCHEMATC

Commit message: wire complete
Parts:
- removed U3: TLV9051, Package_TO_SOT_SMD:SOT-353_SC-70-5, symbol Amplifier_Operational:TLV9001IDCK
- added U3: NCS20071SN, Package_SO:TSOP-5_1.65x3.05mm_P0.95mm, symbol Amplifier_Operational:NCS20071SN
- C1, C2, C3: footprint Capacitor_SMD:C_0402_1005Metric -> Capacitor_SMD:C_0805_2012Metric_Pad1.18x1.45mm_HandSolder
- C4, C5, C6: footprint Capacitor_SMD:C_0402_1005Metric -> Resistor_SMD:R_0805_2012Metric_Pad1.20x1.40mm_HandSolder
- R1, R3: footprint Resistor_SMD:R_0603_1608Metric -> Resistor_SMD:R_0805_2012Metric_Pad1.20x1.40mm_HandSolder
- R10, R11, R12, R13, R14, R15, R16, R17, R18, R19, R2, R4, R5, R6, R7, R8, R9: footprint Resistor_SMD:R_0805_2012Metric -> Resistor_SMD:R_0805_2012Metric_Pad1.20x1.40mm_HandSolder
Connections:
- net +5V: now also U3.5 (V+)
- net ADC: now also U1.10 (PA5_A9_D9_MISO), U3.1; no longer U1.11 (PA6_A10_D10_MOSI)
- net GND: now also U3.2 (V-)
- net S1: now also U1.4 (PA11_A3_D3); no longer U1.2 (PA4_A1_D1)
- net S3: now also U1.2 (PA4_A1_D1); no longer U1.4 (PA11_A3_D3)
- net SENSE: now also U1.11 (PA6_A10_D10_MOSI); no longer U1.10 (PA5_A9_D9_MISO)
- net at R3.1: now also U3.3 (+)
- net at C3.2, R1.1, R2.2: now also U3.4 (-)

Commit message: handsolder pad
Parts:
- U2: footprint Package_TO_SOT_SMD:SOT-23-5 -> Package_TO_SOT_SMD:SOT-23-5_HandSoldering
- U3: footprint Package_SO:TSOP-5_1.65x3.05mm_P0.95mm -> Package_TO_SOT_SMD:SOT-23-5_HandSoldering
Changed lines of the file:
@@
 F 0 "U2" H 1425 2517 50  0000 C CNN
 F 1 "74AHC1G04" H 1425 2426 50  0000 C CNN
-F 2 "Package_TO_SOT_SMD:SOT-23-5" H 1450 2250 50  0001 C CNN
+F 2 "Package_TO_SOT_SMD:SOT-23-5_HandSoldering" H 1450 2250 50  0001 C CNN
 F 3 "http://www.ti.com/lit/sg/scyt129e/scyt129e.pdf" H 1450 2250 50  0001 C CNN
 	1    1450 2250
@@
 F 0 "U3" H 3850 5050 50  0000 L CNN
 F 1 "NCS20071SN" H 3850 4950 50  0000 L CNN
-F 2 "Package_SO:TSOP-5_1.65x3.05mm_P0.95mm" H 3900 6000 50  0001 C CNN
+F 2 "Package_TO_SOT_SMD:SOT-23-5_HandSoldering" H 3900 6000 50  0001 C CNN
 F 3 "https://www.onsemi.com/pub/Collateral/NCS20071-D.PDF" H 3900 6000 50  0001 C CNN
 	1    3850 4800

Commit message: gnd plane
Parts:
- C1, R3: LCSC (none) -> C49678
- C2: LCSC (none) -> C396753
- C3: LCSC (none) -> C157608
- C4, C5, C6: footprint Resistor_SMD:R_0805_2012Metric_Pad1.20x1.40mm_HandSolder -> Capacitor_SMD:C_0805_2012Metric_Pad1.18x1.45mm_HandSolder; LCSC (none) -> C49678
- R1: LCSC (none) -> C115316
- R10, R11, R12, R13, R14, R15, R16, R17, R18, R19, R4, R5, R6, R7, R8, R9: LCSC (none) -> C118844
- R2: LCSC (none) -> C204497
- U2: LCSC (none) -> C7465
- U3: value NCS20071SN -> NCS2003SN2T1G; LCSC (none) -> C89851
- U4, U5: LCSC (none) -> C9386
Changed lines of the file:
@@
 F 2 "Capacitor_SMD:C_0805_2012Metric_Pad1.18x1.45mm_HandSolder" H 3050 4850 50  0001 C CNN
 F 3 "~" H 3050 4850 50  0001 C CNN
+F 4 "C396753" H 3050 4850 50  0001 C CNN "LCSC"
 	1    3050 4850
 	1    0    0    -1
@@
 F 2 "Resistor_SMD:R_0805_2012Metric_Pad1.20x1.40mm_HandSolder" H 3350 4700 50  0001 C CNN
 F 3 "~" H 3350 4700 50  0001 C CNN
+F 4 "C49678" H 3350 4700 50  0001 C CNN "LCSC"
 	1    3350 4700
 	0    1    1    0
@@
 F 2 "Resistor_SMD:R_0805_2012Metric_Pad1.20x1.40mm_HandSolder" H 3850 5500 50  0001 C CNN
 F 3 "~" H 3850 5500 50  0001 C CNN
+F 4 "C204497" H 3850 5500 50  0001 C CNN "LCSC"
 	1    3850 5500
 	0    1    1    0
@@
 F 2 "Resistor_SMD:R_0805_2012Metric_Pad1.20x1.40mm_HandSolder" H 3300 5500 50  0001 C CNN
 F 3 "~" H 3300 5500 50  0001 C CNN
+F 4 "C115316" H 3300 5500 50  0001 C CNN "LCSC"
 	1    3300 5500
 	0    1    1    0
@@
 F 2 "Capacitor_SMD:C_0805_2012Metric_Pad1.18x1.45mm_HandSolder" H 3850 5850 50  0001 C CNN
 F 3 "~" H 3850 5850 50  0001 C CNN
+F 4 "C157608" H 3850 5850 50  0001 C CNN "LCSC"
 	1    3850 5850
 	0    1    1    0
@@
 F 2 "Capacitor_SMD:C_0805_2012Metric_Pad1.18x1.45mm_HandSolder" H 1700 2000 50  0001 C CNN
 F 3 "~" H 1700 2000 50  0001 C CNN
+F 4 "C49678" H 1700 2000 50  0001 C CNN "LCSC"
 	1    1700 2000
 	0    1    1    0
@@
 F 2 "Resistor_SMD:R_0805_2012Metric_Pad1.20x1.40mm_HandSolder" H 6100 5350 50  0001 C CNN
 F 3 "~" H 6100 5350 50  0001 C CNN
+F 4 "C118844" H 6100 5350 50  0001 C CNN "LCSC"
 	1    6100 5350
 	1    0    0    -1
@@
 F 2 "Resistor_SMD:R_0805_2012Metric_Pad1.20x1.40mm_HandSolder" H 6400 5350 50  0001 C CNN
 F 3 "~" H 6400 5350 50  0001 C CNN
+F 4 "C118844" H 6400 5350 50  0001 C CNN "LCSC"
 	1    6400 5350
 	1    0    0    -1
@@
 F 2 "Resistor_SMD:R_0805_2012Metric_Pad1.20x1.40mm_HandSolder" H 6700 5350 50  0001 C CNN
 F 3 "~" H 6700 5350 50  0001 C CNN
+F 4 "C118844" H 6700 5350 50  0001 C CNN "LCSC"
 	1    6700 5350
 	1    0    0    -1
@@
 F 2 "Resistor_SMD:R_0805_2012Metric_Pad1.20x1.40mm_HandSolder" H 7000 5350 50  0001 C CNN
 F 3 "~" H 7000 5350 50  0001 C CNN
+F 4 "C118844" H 7000 5350 50  0001 C CNN "LCSC"
 	1    7000 5350
 	1    0    0    -1
@@
 F 2 "Resistor_SMD:R_0805_2012Metric_Pad1.20x1.40mm_HandSolder" H 7300 5350 50  0001 C CNN
 F 3 "~" H 7300 5350 50  0001 C CNN
+F 4 "C118844" H 7300 5350 50  0001 C CNN "LCSC"
 	1    7300 5350
 	1    0    0    -1
@@
 F 2 "Resistor_SMD:R_0805_2012Metric_Pad1.20x1.40mm_HandSolder" H 7600 5350 50  0001 C CNN
 F 3 "~" H 7600 5350 50  0001 C CNN
+F 4 "C118844" H 7600 5350 50  0001 C CNN "LCSC"
 	1    7600 5350
 	1    0    0    -1
@@
 F 2 "Resistor_SMD:R_0805_2012Metric_Pad1.20x1.40mm_HandSolder" H 7900 5350 50  0001 C CNN
 F 3 "~" H 7900 5350 50  0001 C CNN
+F 4 "C118844" H 7900 5350 50  0001 C CNN "LCSC"
 	1    7900 5350
 	1    0    0    -1
@@
 F 2 "Resistor_SMD:R_0805_2012Metric_Pad1.20x1.40mm_HandSolder" H 8200 5350 50  0001 C CNN
 F 3 "~" H 8200 5350 50  0001 C CNN
+F 4 "C118844" H 8200 5350 50  0001 C CNN "LCSC"
 	1    8200 5350
 	1    0    0    -1
@@
 F 2 "Resistor_SMD:R_0805_2012Metric_Pad1.20x1.40mm_HandSolder" H 8500 5350 50  0001 C CNN
 F 3 "~" H 8500 5350 50  0001 C CNN
+F 4 "C118844" H 8500 5350 50  0001 C CNN "LCSC"
 	1    8500 5350
 	1    0    0    -1
@@
 F 2 "Resistor_SMD:R_0805_2012Metric_Pad1.20x1.40mm_HandSolder" H 8800 5350 50  0001 C CNN
 F 3 "~" H 8800 5350 50  0001 C CNN
+F 4 "C118844" H 8800 5350 50  0001 C CNN "LCSC"
 	1    8800 5350
 	1    0    0    -1
@@
 F 2 "Resistor_SMD:R_0805_2012Metric_Pad1.20x1.40mm_HandSolder" H 9100 5350 50  0001 C CNN
 F 3 "~" H 9100 5350 50  0001 C CNN
+F 4 "C118844" H 9100 5350 50  0001 C CNN "LCSC"
 	1    9100 5350
 	1    0    0    -1
@@
 F 2 "Resistor_SMD:R_0805_2012Metric_Pad1.20x1.40mm_HandSolder" H 9400 5350 50  0001 C CNN
 F 3 "~" H 9400 5350 50  0001 C CNN
+F 4 "C118844" H 9400 5350 50  0001 C CNN "LCSC"
 	1    9400 5350
 	1    0    0    -1
@@
 F 2 "Resistor_SMD:R_0805_2012Metric_Pad1.20x1.40mm_HandSolder" H 9700 5350 50  0001 C CNN
 F 3 "~" H 9700 5350 50  0001 C CNN
+F 4 "C118844" H 9700 5350 50  0001 C CNN "LCSC"
 	1    9700 5350
 	1    0    0    -1
@@
 F 2 "Resistor_SMD:R_0805_2012Metric_Pad1.20x1.40mm_HandSolder" H 10000 5350 50  0001 C CNN
 F 3 "~" H 10000 5350 50  0001 C CNN
+F 4 "C118844" H 10000 5350 50  0001 C CNN "LCSC"
 	1    10000 5350
 	1    0    0    -1
@@
 F 2 "Resistor_SMD:R_0805_2012Metric_Pad1.20x1.40mm_HandSolder" H 10300 5350 50  0001 C CNN
 F 3 "~" H 10300 5350 50  0001 C CNN
+F 4 "C118844" H 10300 5350 50  0001 C CNN "LCSC"
 	1    10300 5350
 	1    0    0    -1
@@
 F 2 "Resistor_SMD:R_0805_2012Metric_Pad1.20x1.40mm_HandSolder" H 10600 5350 50  0001 C CNN
 F 3 "~" H 10600 5350 50  0001 C CNN
+F 4 "C118844" H 10600 5350 50  0001 C CNN "LCSC"
 	1    10600 5350
 	1    0    0    -1
@@
 F 0 "C6" V 1471 5600 50  0000 C CNN
 F 1 "100n" V 1562 5600 50  0000 C CNN
-F 2 "Resistor_SMD:R_0805_2012Metric_Pad1.20x1.40mm_HandSolder" H 1700 5600 50  0001 C CNN
+F 2 "Capacitor_SMD:C_0805_2012Metric_Pad1.18x1.45mm_HandSolder" H 1700 5600 50  0001 C CNN
 F 3 "~" H 1700 5600 50  0001 C CNN
+F 4 "C49678" H 1700 5600 50  0001 C CNN "LCSC"
 	1    1700 5600
 	0    1    1    0
@@
 F 2 "Package_SO:SOIC-16_3.9x9.9mm_P1.27mm" H 1450 6650 50  0001 C CNN
 F 3 "http://www.intersil.com/content/dam/Intersil/documents/cd40/cd4051bms-52bms-53bms.pdf" H 1450 6650 50  0001 C CNN
+F 4 "C9386" H 1450 6650 50  0001 C CNN "LCSC"
 	1    1450 6650
 	1    0    0    -1
@@
 F 0 "C5" V 1471 3050 50  0000 C CNN
 F 1 "100n" V 1562 3050 50  0000 C CNN
-F 2 "Resistor_SMD:R_0805_2012Metric_Pad1.20x1.40mm_HandSolder" H 1700 3050 50  0001 C CNN
+F 2 "Capacitor_SMD:C_0805_2012Metric_Pad1.18x1.45mm_HandSolder" H 1700 3050 50  0001 C CNN
 F 3 "~" H 1700 3050 50  0001 C CNN
+F 4 "C49678" H 1700 3050 50  0001 C CNN "LCSC"
 	1    1700 3050
 	0    1    1    0
@@
 F 2 "Package_SO:SOIC-16_3.9x9.9mm_P1.27mm" H 1450 4100 50  0001 C CNN
 F 3 "http://www.intersil.com/content/dam/Intersil/documents/cd40/cd4051bms-52bms-53bms.pdf" H 1450 4100 50  0001 C CNN
+F 4 "C9386" H 1450 4100 50  0001 C CNN "LCSC"
 	1    1450 4100
 	1    0    0    -1
@@
 F 2 "Package_TO_SOT_SMD:SOT-23-5_HandSoldering" H 1450 2250 50  0001 C CNN
 F 3 "http://www.ti.com/lit/sg/scyt129e/scyt129e.pdf" H 1450 2250 50  0001 C CNN
+F 4 "C7465" H 1450 2250 50  0001 C CNN "LCSC"
 	1    1450 2250
 	1    0    0    -1
@@
 F 0 "C4" V 3771 4350 50  0000 C CNN
 F 1 "100n" V 3862 4350 50  0000 C CNN
-F 2 "Resistor_SMD:R_0805_2012Metric_Pad1.20x1.40mm_HandSolder" H 4000 4350 50  0001 C CNN
+F 2 "Capacitor_SMD:C_0805_2012Metric_Pad1.18x1.45mm_HandSolder" H 4000 4350 50  0001 C CNN
 F 3 "~" H 4000 4350 50  0001 C CNN
+F 4 "C49678" H 4000 4350 50  0001 C CNN "LCSC"
 	1    4000 4350
 	0    1    1    0
@@
 P 3850 4800
 F 0 "U3" H 3850 5050 50  0000 L CNN
-F 1 "NCS20071SN" H 3850 4950 50  0000 L CNN
+F 1 "NCS2003SN2T1G" H 3850 4950 50  0000 L CNN
 F 2 "Package_TO_SOT_SMD:SOT-23-5_HandSoldering" H 3900 6000 50  0001 C CNN
-F 3 "https://www.onsemi.com/pub/Collateral/NCS20071-D.PDF" H 3900 6000 50  0001 C CNN
+F 3 "https://www.onsemi.com/pdf/datasheet/ncs2003-d.pdf" H 3900 6000 50  0001 C CNN
+F 4 "C89851" H 3850 4800 50  0001 C CNN "LCSC"
 	1    3850 4800
 	1    0    0    -1

Commit message: trace adjust
Parts:
- renumbered SW9 to SW4
Connections:
- net col1: now also SW4.2
- net col2: no longer SW4.2
Other:
- moved on the sheet: SW4
Changed lines of the file:
@@
 $EndComp
 $Comp
-L ec_sw:EC_SW SW9
+L ec_sw:EC_SW SW4
 U 1 1 619757AB
-P 6250 4300
-F 0 "SW9" H 6283 4515 50  0000 C CNN
-F 1 "LSHFT" H 6283 4424 50  0000 C CNN
-F 2 "lib:ecs_pad" H 6250 4050 50  0001 C CNN
-F 3 "" H 6250 4050 50  0000 C CNN
-	1    6250 4300
+P 5950 4300
+F 0 "SW4" H 5983 4515 50  0000 C CNN
+F 1 "LSHFT" H 5983 4424 50  0000 C CNN
+F 2 "lib:ecs_pad" H 5950 4050 50  0001 C CNN
+F 3 "" H 5950 4050 50  0000 C CNN
+	1    5950 4300
 	1    0    0    -1
 $EndComp
@@
 L power:GND #PWR0120
 U 1 1 619757B1
-P 6300 4400
-F 0 "#PWR0120" H 6300 4150 50  0001 C CNN
-F 1 "GND" H 6305 4227 50  0001 C CNN
-F 2 "" H 6300 4400 50  0001 C CNN
-F 3 "" H 6300 4400 50  0001 C CNN
-	1    6300 4400
+P 6000 4400
+F 0 "#PWR0120" H 6000 4150 50  0001 C CNN
+F 1 "GND" H 6005 4227 50  0001 C CNN
+F 2 "" H 6000 4400 50  0001 C CNN
+F 3 "" H 6000 4400 50  0001 C CNN
+	1    6000 4400
 	1    0    0    -1
 $EndComp
@@
 	6400 2650 6400 3200
 Connection ~ 6400 3200
-Connection ~ 6400 4300
-Wire Wire Line
-	6400 4300 6400 4850
 $Comp
 L ec_sw:EC_SW SW11
@@
 $EndComp
 $Comp
-L ec_sw:EC_SW SW48
-U 1 1 619EA77A
-P 8650 3750
-F 0 "SW48" H 8683 3965 50  0000 C CNN
-F 1 "L" H 8683 3874 50  0000 C CNN
-F 2 "lib:ecs_pad" H 8650 3500 50  0001 C CNN
-F 3 "" H 8650 3500 50  0000 C CNN
-	1    8650 3750
-	1    0    0    -1
-$EndComp
-$Comp
 L power:GND #PWR0159
 U 1 1 619EA780
@@
 	8600 4000 8900 4000
 Connection ~ 8900 4000
-Wire Wire Line
-	8900 4000 9200 4000
 Connection ~ 9200 4000
 Connection ~ 9800 4000
-Connection ~ 6200 4550
-Wire Wire Line
-	6200 4550 6500 4550
 Connection ~ 6500 4550
 Wire Wire Line
@@
 	10100 5100 10400 5100
 Wire Wire Line
-	5750 4550 6200 4550
-Wire Wire Line
-	6100 3750 6100 4850
-Wire Wire Line
-	6400 3200 6400 3750
+	5750 4550 5900 4550
+Wire Wire Line
+	6100 3750 6100 4300
 Wire Wire Line
 	6200 5100 6800 5100
@@
 	2350 3500 1950 3500
 Connection ~ 2350 4700
-$Comp
-L ec_sw:EC_SW SW8
-U 1 1 61988E43
-P 6250 3750
-F 0 "SW8" H 6283 3965 50  0000 C CNN
-F 1 "A" H 6283 3874 50  0000 C CNN
-F 2 "lib:ecs_pad" H 6250 3500 50  0001 C CNN
-F 3 "" H 6250 3500 50  0000 C CNN
-	1    6250 3750
-	1    0    0    -1
-$EndComp
 Wire Wire Line
 	6700 3200 6700 3750
-Wire Wire Line
-	5900 4000 6200 4000
 $Comp
 L power:GND #PWR0186
@@
 Wire Wire Line
 	6700 3750 6700 4300
-Connection ~ 6200 4000
-Wire Wire Line
-	6200 4000 6500 4000
-Connection ~ 6400 3750
-Wire Wire Line
-	6400 3750 6400 4300
-Wire Wire Line
-	9200 4000 9800 4000
-Wire Wire Line
-	9700 3200 9700 4850
+Wire Wire Line
+	9200 4000 9500 4000
+Wire Wire Line
+	9700 3200 9700 3750
 $Comp
 L power:GND #PWR0104
@@
 	1    0    0    -1
 $EndComp
+Connection ~ 5900 4550
+Connection ~ 6100 4300
+Wire Wire Line
+	6100 4300 6100 4850
+Wire Wire Line
+	5900 4550 6500 4550
+$Comp
+L ec_sw:EC_SW SW8
+U 1 1 61988E43
+P 6250 3750
+F 0 "SW8" H 6283 3965 50  0000 C CNN
+F 1 "A" H 6283 3874 50  0000 C CNN
+F 2 "lib:ecs_pad" H 6250 3500 50  0001 C CNN
+F 3 "" H 6250 3500 50  0000 C CNN
+	1    6250 3750
+	1    0    0    -1
+$EndComp
+Connection ~ 9500 4000
+Wire Wire Line
+	9500 4000 9800 4000
+Connection ~ 9700 3750
+Wire Wire Line
+	9700 3750 9700 4850
+Wire Wire Line
+	8900 4000 9200 4000
+$Comp
+L ec_sw:EC_SW SW48
+U 1 1 619EA77A
+P 8650 3750
+F 0 "SW48" H 8683 3965 50  0000 C CNN
+F 1 "L" H 8683 3874 50  0000 C CNN
+F 2 "lib:ecs_pad" H 8650 3500 50  0001 C CNN
+F 3 "" H 8650 3500 50  0000 C CNN
+	1    8650 3750
+	1    0    0    -1
+$EndComp
+Wire Wire Line
+	6400 3200 6400 3750
+Wire Wire Line
+	5900 4000 6200 4000
+Connection ~ 6200 4000
+Wire Wire Line
+	6200 4000 6500 4000
+Connection ~ 6400 3750
+Wire Wire Line
+	6400 3750 6400 4850
 $EndSCHEMATC
