File: pcb/tc69.kicad_sch (KiCad schematic)
At the start: 98 parts, among them SW1 ESC, SW10 LWIN, SW11 2, SW12 W, SW13 S, SW14 Z, SW16 3, SW17 E, SW18 D, SW19 X, SW2 TAB, SW20 LALT, SW21 4, SW22 R, SW23 F, SW24 C, SW26 5, SW27 T, SW28 G, SW29 V, SW3 CAPS, SW30 LSPC, SW31 6, SW32 Y, SW33 H, SW34 B, SW36 7, SW37 U, SW38 J, SW39 N, SW4 LSHFT, SW41 8, SW42 I, SW43 K, SW44 M, SW45 RSPC, SW46 9, SW47 O, SW48 L, SW49 COMMA, SW5 LCTRL, SW51 0, SW52 P, SW53 SCLN, SW54 DOT, SW55 RALT, SW56 MINUS, SW57 LBRC, SW58 QUOTE, SW59 SLSH, SW6 1, SW60 RWIN, SW61 EQUAL, SW62 RBRC, SW65 APP, SW66 BS, SW68 ENTER, SW69 RSHFT, SW7 Q, SW70 LEFT, SW72 BSLSH, SW74 UP, SW75 DOWN, SW76 HOME, SW77 PGUP, SW78 PGDN, SW79 END, SW8 A, SW80 RIGHT, U1 SeeeduinoXIAO, U2 74AHC1G04, U3 NCS2003SN2T1G, U4 4051, U5 4051

Commit message: jlcpcb r2
Parts:
- U3: value NCS2003SN2T1G -> AD8601ARTZ
Connections:
- net S2: now also U1.5 (PA8_A4_D4_SDA); no longer U1.10 (PA5_A9_D9_MISO)
- net row1: now also U1.9 (PA7_A8_D8_SCK); no longer U1.8 (PB09_A7_D7_RX)
- net row2: now also U1.10 (PA5_A9_D9_MISO); no longer U1.9 (PA7_A8_D8_SCK)
- net row3: now also U1.8 (PB09_A7_D7_RX); no longer U1.7 (PB08_A6_D6_TX)
- net row4: now also U1.7 (PB08_A6_D6_TX); no longer U1.6 (PA9_A5_D5_SCL)
- net row5: now also U1.6 (PA9_A5_D5_SCL); no longer U1.5 (PA8_A4_D4_SDA)
Changed lines of the file:
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@@
     (stroke (width 0) (type default) (color 0 0 0 0))
   )
-  (global_label "row5" (shape input) (at 87.63 49.53 180) (fields_autoplaced)
+  (global_label "row5" (shape input) (at 87.63 53.34 180) (fields_autoplaced)
     (effects (font (size 1.27 1.27)) (justify right))
-    (property "Intersheet References" "${INTERSHEET_REFS}" (id 0) (at 0 0 0)
+    (property "Intersheet References" "${INTERSHEET_REFS}" (id 0) (at 0 3.81 0)
       (effects (font (size 1.27 1.27)) hide)
     )
@@
     )
   )
-  (global_label "row3" (shape input) (at 87.63 57.15 180) (fields_autoplaced)
-    (effects (font (size 1.27 1.27)) (justify right))
-    (property "Intersheet References" "${INTERSHEET_REFS}" (id 0) (at 0 0 0)
+  (global_label "row3" (shape input) (at 129.54 57.15 0) (fields_autoplaced)
+    (effects (font (size 1.27 1.27)) (justify left))
+    (property "Intersheet References" "${INTERSHEET_REFS}" (id 0) (at 217.17 114.3 0)
       (effects (font (size 1.27 1.27)) hide)
     )
@@
     )
   )
-  (global_label "row1" (shape input) (at 129.54 57.15 0) (fields_autoplaced)
+  (global_label "row1" (shape input) (at 129.54 53.34 0) (fields_autoplaced)
     (effects (font (size 1.27 1.27)) (justify left))
-    (property "Intersheet References" "${INTERSHEET_REFS}" (id 0) (at 0 0 0)
+    (property "Intersheet References" "${INTERSHEET_REFS}" (id 0) (at 0 -3.81 0)
       (effects (font (size 1.27 1.27)) hide)
     )
@@
     )
   )
-  (global_label "row2" (shape input) (at 129.54 53.34 0) (fields_autoplaced)
+  (global_label "row2" (shape input) (at 129.54 49.53 0) (fields_autoplaced)
     (effects (font (size 1.27 1.27)) (justify left))
-    (property "Intersheet References" "${INTERSHEET_REFS}" (id 0) (at 0 0 0)
+    (property "Intersheet References" "${INTERSHEET_REFS}" (id 0) (at 0 -3.81 0)
       (effects (font (size 1.27 1.27)) hide)
     )
@@
     )
   )
-  (global_label "S2" (shape input) (at 129.54 49.53 0) (fields_autoplaced)
-    (effects (font (size 1.27 1.27)) (justify left))
-    (property "Intersheet References" "${INTERSHEET_REFS}" (id 0) (at 0 0 0)
+  (global_label "S2" (shape input) (at 87.63 49.53 180) (fields_autoplaced)
+    (effects (font (size 1.27 1.27)) (justify right))
+    (property "Intersheet References" "${INTERSHEET_REFS}" (id 0) (at 217.17 99.06 0)
       (effects (font (size 1.27 1.27)) hide)
     )
@@
     )
   )
-  (global_label "row4" (shape input) (at 87.63 53.34 180) (fields_autoplaced)
+  (global_label "row4" (shape input) (at 87.63 57.15 180) (fields_autoplaced)
     (effects (font (size 1.27 1.27)) (justify right))
-    (property "Intersheet References" "${INTERSHEET_REFS}" (id 0) (at 0 0 0)
+    (property "Intersheet References" "${INTERSHEET_REFS}" (id 0) (at 0 3.81 0)
       (effects (font (size 1.27 1.27)) hide)
     )
@@
       (effects (font (size 1.27 1.27)) (justify left))
     )
-    (property "Value" "NCS2003SN2T1G" (id 1) (at 97.79 118.11 0)
+    (property "Value" "AD8601ARTZ" (id 1) (at 97.79 118.11 0)
       (effects (font (size 1.27 1.27)) (justify left))
     )
@@
     )
     (path "/00000000-0000-0000-0000-0000619b1295"
-      (reference "U3") (unit 1) (value "NCS2003SN2T1G") (footprint "Package_TO_SOT_SMD:SOT-23-5_HandSoldering")
+      (reference "U3") (unit 1) (value "AD8601ARTZ") (footprint "Package_TO_SOT_SMD:SOT-23-5_HandSoldering")
     )
     (path "/00000000-0000-0000-0000-000061a21e5a"

Commit message: add keepout on F_Cu
Parts:
- SW1, SW10, SW11, SW12, SW13, SW14, SW16, SW17, SW18, SW19, SW2, SW20, SW21, SW22, SW23, SW24, SW26, SW27, SW28, SW29, SW3, SW30, SW31, SW32, SW33, SW34, SW36, SW37, SW38, SW39, SW4, SW41, SW42, SW43, SW44, SW45, SW46, SW47, SW48, SW49, SW5, SW51, SW52, SW53, SW54, SW55, SW56, SW57, SW58, SW59, SW6, SW60, SW61, SW62, SW65, SW66, SW68, SW69, SW7, SW70, SW72, SW74, SW75, SW76, SW77, SW78, SW79, SW8, SW80: footprint lib:ecs_pad -> CapacitivePad:CapacitivePad

Commit message: revert to the rp2040 version
Parts:
- C2: footprint Capacitor_SMD:C_0805_2012Metric_Pad1.18x1.45mm_HandSolder -> Capacitor_SMD:C_0603_1608Metric_Pad1.08x0.95mm_HandSolder
- SW1, SW10, SW11, SW12, SW13, SW14, SW16, SW17, SW18, SW19, SW2, SW20, SW21, SW22, SW23, SW24, SW26, SW27, SW28, SW29, SW3, SW30, SW31, SW32, SW33, SW34, SW36, SW37, SW38, SW39, SW4, SW41, SW42, SW43, SW44, SW45, SW46, SW47, SW48, SW49, SW5, SW51, SW52, SW53, SW54, SW55, SW56, SW57, SW58, SW59, SW6, SW60, SW61, SW62, SW65, SW66, SW68, SW69, SW7, SW70, SW72, SW74, SW75, SW76, SW77, SW78, SW79, SW8, SW80: footprint CapacitivePad:CapacitivePad -> lib:ecs_pad
